Commit message: Got the simulation running with ros2_control

File: src/description/urdf/links.urdf.xacro (robot description, xacro)
@@ -35,5 +35,5 @@
         </collision>
         <xacro:inertial_cylinder mass="0.1" length="0.04" radius="0.05">
-            <origin xyz="0 0 0" rpy="0 0 0"/>
+            <origin xyz="0 0 0" rpy="0 0 0" />
         </xacro:inertial_cylinder>
     </link>
@@ -51,5 +51,5 @@
         </collision>
         <xacro:inertial_cylinder mass="0.1" length="0.04" radius="0.05">
-            <origin xyz="0 0 0" rpy="0 0 0"/>
+            <origin xyz="0 0 0" rpy="0 0 0" />
         </xacro:inertial_cylinder>
     </link>
@@ -67,6 +67,20 @@
         </collision>
         <xacro:inertial_sphere mass="0.1" radius="0.05">
-            <origin xyz="0 0 0" rpy="0 0 0"/>
+            <origin xyz="0 0 0" rpy="0 0 0" />
         </xacro:inertial_sphere>
     </link>
+    <gazebo reference="chassis_link">
+        <material>Gazebo/SkyBlue</material>
+    </gazebo>
+    <gazebo reference="right_wheel_link">
+        <material>Gazebo/Black</material>
+    </gazebo>
+    <gazebo reference="left_wheel_link">
+        <material>Gazebo/Black</material>
+    </gazebo>
+    <gazebo reference="caster_link">
+        <material>Gazebo/Grey</material>
+        <mu1 value="0.001" />
+        <mu2 value="0.001" />
+    </gazebo>
 </robot>

File: src/description/urdf/materials.urdf.xacro (robot description, xacro)
@@ -13,3 +13,6 @@
         <color rgba="0 0 0 1" />
     </material>
+    <material name="red">
+        <color rgba="1 0 0 1" />
+    </material>
 </robot>

File: src/description/urdf/robot.urdf.xacro (robot description, xacro)
@@ -2,4 +2,9 @@
 <robot name="robot" xmlns:xacro="http://www.ros.org/wiki/xacro">
     <xacro:include filename="links.urdf.xacro" />
+    <xacro:include filename="lidar.urdf.xacro" />
+    <!-- <xacro:include filename="camera.urdf.xacro" /> -->
+    <xacro:include filename="depth_camera.urdf.xacro" />
     <xacro:include filename="joints.urdf.xacro" />
+    <!-- <xacro:include filename="gazebo_control.xacro" /> -->
+    <xacro:include filename="ros2_control.xacro" />
 </robot>
