Commit message: Add inertia and gazebo tags, entity spawns successfully in gazebo

File: src/diff_bot/urdf/links.urdf.xacro (robot description, xacro)
@@ -1,4 +1,6 @@
 <?xml version="1.0"?>
 <robot name="ultron" xmlns:xacro="http://www.ros.org/wiki/xacro">
+    <xacro:include filename="materials.xacro" />
+    <xacro:include filename="inertia_macros.xacro" />
     <link name="base_link" />
     <link name="chassis_link">
@@ -8,7 +10,5 @@
                 <mesh filename="file://$(find diff_bot)/mesh/Chassis.stl" />
             </geometry>
-            <material name="blue">
-                <color rgba="0 0 1 1" />
-            </material>
+            <material name="blue" />
         </visual>
         <collision>
@@ -18,5 +18,13 @@
             </geometry>
         </collision>
+        <xacro:inertial_cuboid mass="3.5" x="0.3" y="0.25" z="0.05">
+            <origin xyz="0 0 0" rpy="0 0 0" />
+        </xacro:inertial_cuboid>
     </link>
+    <gazebo reference="chassis_link">
+        <material>Gazebo/Turquoise</material>
+        <mu1 value="0.01" />
+        <mu2 value="0.02" />
+    </gazebo>
     <link name="right_wheel_link">
         <visual>
@@ -25,7 +33,5 @@
                 <mesh filename="file://$(find diff_bot)/mesh/Wheel.stl" />
             </geometry>
-            <material name="grey">
-                <color rgba="0.2 0.2 0.2 1" />
-            </material>
+            <material name="grey" />
         </visual>
         <collision>
@@ -35,5 +41,11 @@
             </geometry>
         </collision>
+        <xacro:inertial_cylinder mass="0.05" radius="0.025" length="0.017">
+            <origin xyz="0 0 0" rpy="0 0 0" />
+        </xacro:inertial_cylinder>
     </link>
+    <gazebo reference="right_wheel_link">
+        <material>Gazebo/Grey</material>
+    </gazebo>
     <link name="left_wheel_link">
         <visual>
@@ -42,7 +54,5 @@
                 <mesh filename="file://$(find diff_bot)/mesh/Wheel.stl" />
             </geometry>
-            <material name="grey">
-                <color rgba="0.2 0.2 0.2 1" />
-            </material>
+            <material name="grey" />
         </visual>
         <collision>
@@ -52,4 +62,10 @@
             </geometry>
         </collision>
+        <xacro:inertial_cylinder mass="0.05" radius="0.025" length="0.017">
+            <origin xyz="0 0 0" rpy="0 0 0" />
+        </xacro:inertial_cylinder>
     </link>
+    <gazebo reference="left_wheel_link">
+        <material>Gazebo/Grey</material>
+    </gazebo>
 </robot>
