Commit message: Bug found: PointCLoud rotates to opposite direction

File: src/diff_bot/urdf/joints.urdf.xacro (robot description, xacro)
@@ -3,10 +3,10 @@
     <joint name="chassis_joint" type="fixed">
         <parent link="base_link" />
-        <child link="chassis" />
+        <child link="chassis_link" />
         <origin xyz="0 0 0.017" rpy="0 0 0" />
     </joint>
     <joint name="right_wheel_joint" type="continuous">
-        <parent link="chassis" />
-        <child link="right_wheel" />
+        <parent link="chassis_link" />
+        <child link="right_wheel_link" />
         <origin xyz="-0.067 -0.082 0.008" rpy="0 0 0" />
         <limits effort="10" velocity="10" />
@@ -14,6 +14,6 @@
     </joint>
     <joint name="left_wheel_joint" type="continuous">
-        <parent link="chassis" />
-        <child link="left_wheel" />
+        <parent link="chassis_link" />
+        <child link="left_wheel_link" />
         <origin xyz="-0.067 0.082 0.008" rpy="0 0 ${pi}" />
         <limits effort="10" velocity="10" />
@@ -21,12 +21,17 @@
     </joint>
     <joint name="lidar_joint" type="fixed">
-        <parent link="chassis" />
-        <child link="lidar" />
+        <parent link="chassis_link" />
+        <child link="lidar_link" />
         <origin xyz="0 0 0.065" rpy="0 0 0" />
     </joint>
     <joint name="camera_joint" type="fixed">
-        <parent link="chassis" />
-        <child link="camera" />
+        <parent link="chassis_link" />
+        <child link="camera_link" />
         <origin xyz="0.1 0 0.02" rpy="0 0 0" />
     </joint>
+    <joint name="camera_sensor_joint" type="fixed">
+        <parent link="camera_link" />
+        <child link="camera_sensor_link" />
+        <origin xyz="0 0 0" rpy="${-pi / 2} 0 ${-pi / 2}" />
+    </joint>
 </robot>

File: src/diff_bot/urdf/links.urdf.xacro (robot description, xacro)
@@ -4,5 +4,5 @@
     <xacro:include filename="inertia_macros.xacro" />
     <link name="base_link" />
-    <link name="chassis">
+    <link name="chassis_link">
         <visual>
             <origin xyz="0 0 0" rpy="0 0 0" />
@@ -22,10 +22,10 @@
         </xacro:inertial_cuboid>
     </link>
-    <gazebo reference="chassis">
+    <gazebo reference="chassis_link">
         <mu1 value="0.001" />
         <mu2 value="0.001" />
         <material>Gazebo/Blue</material>
     </gazebo>
-    <link name="right_wheel">
+    <link name="right_wheel_link">
         <visual>
             <origin xyz="0 0 0" rpy="0 0 0" />
@@ -45,8 +45,8 @@
         </xacro:inertial_cylinder>
     </link>
-    <gazebo reference="right_wheel">
+    <gazebo reference="right_wheel_link">
         <material>Gazebo/Black</material>
     </gazebo>
-    <link name="left_wheel">
+    <link name="left_wheel_link">
         <visual>
             <origin xyz="0 0 0" rpy="0 0 0" />
@@ -66,8 +66,8 @@
         </xacro:inertial_cylinder>
     </link>
-    <gazebo reference="left_wheel">
+    <gazebo reference="left_wheel_link">
         <material>Gazebo/Black</material>
     </gazebo>
-    <link name="lidar">
+    <link name="lidar_link">
         <visual>
             <origin xyz="0 0 0" rpy="0 0 0" />
@@ -87,8 +87,8 @@
         </xacro:inertial_cylinder>
     </link>
-    <gazebo reference="lidar">
+    <gazebo reference="lidar_link">
         <material>Gazebo/Orange</material>
     </gazebo>
-    <link name="camera">
+    <link name="camera_link">
         <visual>
             <origin xyz="-0.007 0 0" rpy="0 0 0" />
@@ -108,6 +108,7 @@
         </xacro:inertial_cuboid>
     </link>
-    <gazebo reference="camera">
+    <gazebo reference="camera_link">
         <material>Gazebo/Red</material>
     </gazebo>
+    <link name="camera_sensor_link" />
 </robot>

File: src/diff_bot/urdf/robot.urdf.xacro (robot description, xacro)
@@ -3,3 +3,4 @@
     <xacro:include filename="links.urdf.xacro" />
     <xacro:include filename="joints.urdf.xacro" />
+    <xacro:include filename="gazebo_sensors.xacro" />
 </robot>

Commit message: Checkpoint: Add rsp.launch.py

File: src/diff_bot/urdf/joints.urdf.xacro (robot description, xacro)
@@ -1,4 +1,4 @@
 <?xml version="1.0"?>
-<robot name="diff_bot" xmlns:xacro="http://www.ros.org/wiki/xacro">
+<robot name="ultron" xmlns:xacro="http://www.ros.org/wiki/xacro">
     <joint name="chassis_joint" type="fixed">
         <parent link="base_link" />
@@ -6,32 +6,13 @@
         <origin xyz="0 0 0.017" rpy="0 0 0" />
     </joint>
-    <joint name="right_wheel_joint" type="continuous">
+    <joint name="right_wheel_joint" type="fixed">
         <parent link="chassis_link" />
         <child link="right_wheel_link" />
-        <origin xyz="-0.067 -0.082 0.008" rpy="0 0 0" />
-        <limits effort="10" velocity="10" />
-        <axis xyz="0 1 0" />
+        <origin xyz="-0.067 -0.089 0.008" rpy="0 0 0" />
     </joint>
-    <joint name="left_wheel_joint" type="continuous">
+    <joint name="left_wheel_joint" type="fixed">
         <parent link="chassis_link" />
         <child link="left_wheel_link" />
-        <origin xyz="-0.067 0.082 0.008" rpy="0 0 ${pi}" />
-        <limits effort="10" velocity="10" />
-        <axis xyz="0 -1 0" />
-    </joint>
-    <joint name="lidar_joint" type="fixed">
-        <parent link="chassis_link" />
-        <child link="lidar_link" />
-        <origin xyz="0 0 0.065" rpy="0 0 0" />
-    </joint>
-    <joint name="camera_joint" type="fixed">
-        <parent link="chassis_link" />
-        <child link="camera_link" />
-        <origin xyz="0.1 0 0.02" rpy="0 0 0" />
-    </joint>
-    <joint name="camera_sensor_joint" type="fixed">
-        <parent link="camera_link" />
-        <child link="camera_sensor_link" />
-        <origin xyz="0 0 0" rpy="${-pi / 2} 0 ${-pi / 2}" />
+        <origin xyz="-0.067 0.089 0.008" rpy="0 0 0" />
     </joint>
 </robot>

File: src/diff_bot/urdf/links.urdf.xacro (robot description, xacro)
@@ -1,6 +1,4 @@
 <?xml version="1.0"?>
-<robot name="diff_bot" xmlns:xacro="http://www.ros.org/wiki/xacro">
-    <xacro:include filename="materials.xacro" />
-    <xacro:include filename="inertia_macros.xacro" />
+<robot name="ultron" xmlns:xacro="http://www.ros.org/wiki/xacro">
     <link name="base_link" />
     <link name="chassis_link">
@@ -8,107 +6,50 @@
             <origin xyz="0 0 0" rpy="0 0 0" />
             <geometry>
-                <mesh filename="file://$(find diff_bot)/meshes/Chassis.stl" />
+                <mesh filename="file://$(find diff_bot)/mesh/Chassis.stl" />
             </geometry>
-            <material name="blue" />
+            <material name="blue">
+                <color rgba="0 0 1 1" />
+            </material>
         </visual>
         <collision>
             <origin xyz="0 0 0" rpy="0 0 0" />
             <geometry>
-                <mesh filename="file://$(find diff_bot)/meshes/Chassis.stl" />
+                <mesh filename="file://$(find diff_bot)/mesh/Chassis.stl" />
             </geometry>
         </collision>
-        <xacro:inertial_cuboid mass="1.4" x="0.15" y="0.2" z="0.07">
-            <origin xyz="0 0 0" rpy="0 0 0" />
-        </xacro:inertial_cuboid>
     </link>
-    <gazebo reference="chassis_link">
-        <mu1 value="0.001" />
-        <mu2 value="0.001" />
-        <material>Gazebo/Blue</material>
-    </gazebo>
     <link name="right_wheel_link">
         <visual>
             <origin xyz="0 0 0" rpy="0 0 0" />
             <geometry>
-                <mesh filename="file://$(find diff_bot)/meshes/Wheel.stl" />
+                <mesh filename="file://$(find diff_bot)/mesh/Wheel.stl" />
             </geometry>
-            <material name="black" />
+            <material name="grey">
+                <color rgba="0.2 0.2 0.2 1" />
+            </material>
         </visual>
         <collision>
             <origin xyz="0 0 0" rpy="0 0 0" />
             <geometry>
-                <mesh filename="file://$(find diff_bot)/meshes/Wheel.stl" />
+                <mesh filename="file://$(find diff_bot)/mesh/Wheel.stl" />
             </geometry>
         </collision>
-        <xacro:inertial_cylinder mass="0.02" radius="0.025" length="0.015">
-            <origin xyz="0 0 0" rpy="0 0 0" />
-        </xacro:inertial_cylinder>
     </link>
-    <gazebo reference="right_wheel_link">
-        <material>Gazebo/Black</material>
-    </gazebo>
     <link name="left_wheel_link">
         <visual>
             <origin xyz="0 0 0" rpy="0 0 0" />
             <geometry>
-                <mesh filename="file://$(find diff_bot)/meshes/Wheel.stl" />
+                <mesh filename="file://$(find diff_bot)/mesh/Wheel.stl" />
             </geometry>
-            <material name="black" />
+            <material name="grey">
+                <color rgba="0.2 0.2 0.2 1" />
+            </material>
         </visual>
         <collision>
             <origin xyz="0 0 0" rpy="0 0 0" />
             <geometry>
-                <mesh filename="file://$(find diff_bot)/meshes/Wheel.stl" />
+                <mesh filename="file://$(find diff_bot)/mesh/Wheel.stl" />
             </geometry>
         </collision>
-        <xacro:inertial_cylinder mass="0.02" radius="0.025" length="0.015">
-            <origin xyz="0 0 0" rpy="0 0 0" />
-        </xacro:inertial_cylinder>
     </link>
-    <gazebo reference="left_wheel_link">
-        <material>Gazebo/Black</material>
-    </gazebo>
-    <link name="lidar_link">
-        <visual>
-            <origin xyz="0 0 0" rpy="0 0 0" />
-            <geometry>
-                <mesh filename="file://$(find diff_bot)/meshes/Lidar.stl" />
-            </geometry>
-            <material name="orange" />
-        </visual>
-        <collision>
-            <origin xyz="0 0 0" rpy="0 0 0" />
-            <geometry>
-                <mesh filename="file://$(find diff_bot)/meshes/Lidar.stl" />
-            </geometry>
-        </collision>
-        <xacro:inertial_cylinder mass="0.08" radius="0.035" length="0.025">
-            <origin xyz="0 0 0" rpy="0 0 0" />
-        </xacro:inertial_cylinder>
-    </link>
-    <gazebo reference="lidar_link">
-        <material>Gazebo/Orange</material>
-    </gazebo>
-    <link name="camera_link">
-        <visual>
-            <origin xyz="-0.007 0 0" rpy="0 0 0" />
-            <geometry>
-                <mesh filename="file://$(find diff_bot)/meshes/Camera.stl" />
-            </geometry>
-            <material name="red" />
-        </visual>
-        <collision>
-            <origin xyz="-0.007 0 0" rpy="0 0 0" />
-            <geometry>
-                <mesh filename="file://$(find diff_bot)/meshes/Camera.stl" />
-            </geometry>
-        </collision>
-        <xacro:inertial_cuboid mass="0.3" x="0.007" y="0.02" z="0.015">
-            <origin xyz="0 0 0" rpy="0 0 0" />
-        </xacro:inertial_cuboid>
-    </link>
-    <gazebo reference="camera_link">
-        <material>Gazebo/Red</material>
-    </gazebo>
-    <link name="camera_sensor_link" />
 </robot>

File: src/diff_bot/urdf/robot.urdf.xacro (robot description, xacro)
@@ -1,6 +1,5 @@
 <?xml version="1.0"?>
-<robot name="diff_bot" xmlns:xacro="http://www.ros.org/wiki/xacro">
+<robot name="ultron" xmlns:xacro="http://www.ros.org/wiki/xacro">
     <xacro:include filename="links.urdf.xacro" />
     <xacro:include filename="joints.urdf.xacro" />
-    <xacro:include filename="gazebo_sensors.xacro" />
 </robot>

Commit message: Checkpoint: Add sim.launch.py

File: src/diff_bot/urdf/joints.urdf.xacro (robot description, xacro)
@@ -6,13 +6,15 @@
         <origin xyz="0 0 0.017" rpy="0 0 0" />
     </joint>
-    <joint name="right_wheel_joint" type="fixed">
+    <joint name="right_wheel_joint" type="continuous">
         <parent link="chassis_link" />
         <child link="right_wheel_link" />
         <origin xyz="-0.067 -0.089 0.008" rpy="0 0 0" />
+        <axis xyz="0 1 0" />
     </joint>
-    <joint name="left_wheel_joint" type="fixed">
+    <joint name="left_wheel_joint" type="continuous">
         <parent link="chassis_link" />
         <child link="left_wheel_link" />
         <origin xyz="-0.067 0.089 0.008" rpy="0 0 0" />
+        <axis xyz="0 1 0" />
     </joint>
 </robot>

Commit message: Add lidar link and plugin

File: src/diff_bot/urdf/joints.urdf.xacro (robot description, xacro)
@@ -18,3 +18,8 @@
         <axis xyz="0 1 0" />
     </joint>
+    <joint name="lidar_joint" type="fixed">
+        <parent link="chassis_link" />
+        <child link="lidar_link" />
+        <origin xyz="0 0 0.0775" rpy="0 0 0" />
+    </joint>
 </robot>

File: src/diff_bot/urdf/links.urdf.xacro (robot description, xacro)
@@ -69,3 +69,22 @@
         <material>Gazebo/Grey</material>
     </gazebo>
+    <link name="lidar_link">
+        <visual>
+            <geometry>
+                <mesh filename="file://$(find diff_bot)/mesh/Lidar.stl" />
+            </geometry>
+            <material name="purple" />
+        </visual>
+        <collision>
+            <geometry>
+                <mesh filename="file://$(find diff_bot)/mesh/Lidar.stl" />
+            </geometry>
+        </collision>
+        <xacro:inertial_cylinder mass="0.1" radius="0.0375" length="0.025">
+            <origin xyz="0 0 0" rpy="0 0 0" />
+        </xacro:inertial_cylinder>
+    </link>
+    <gazebo reference="lidar_link">
+        <material>Gazebo/Purple</material>
+    </gazebo>
 </robot>

File: src/diff_bot/urdf/materials.xacro (robot description, xacro)
@@ -19,3 +19,6 @@
         <color rgba="1 0 0 1" />
     </material>
+    <material name="purple">
+        <color rgba="1 0 1 1" />
+    </material>
 </robot>

File: src/diff_bot/urdf/robot.urdf.xacro (robot description, xacro)
@@ -4,3 +4,4 @@
     <xacro:include filename="joints.urdf.xacro" />
     <xacro:include filename="diff_control.gazebo.xacro" />
+    <xacro:include filename="lidar.gazebo.xacro" />
 </robot>
