Commit message: SLAM done except map does not load on startup

File: src/diff_bot/urdf/diff_control.gazebo.xacro (robot description, xacro)
@@ -10,5 +10,5 @@
             <max_wheel_acceleration>4</max_wheel_acceleration>
             <odometry_frame>odom</odometry_frame>
-            <ros_base_frame>base_link</ros_base_frame>
+            <ros_base_frame>base_footprint</ros_base_frame>
             <publish_odom>true</publish_odom>
             <publish_odom_tf>true</publish_odom_tf>

File: src/diff_bot/urdf/joints.urdf.xacro (robot description, xacro)
@@ -2,5 +2,5 @@
 <robot name="ultron" xmlns:xacro="http://www.ros.org/wiki/xacro">
     <joint name="chassis_joint" type="fixed">
-        <parent link="base_link" />
+        <parent link="base_footprint" />
         <child link="chassis_link" />
         <origin xyz="0 0 0.017" rpy="0 0 0" />

File: src/diff_bot/urdf/lidar.gazebo.xacro (robot description, xacro)
@@ -4,5 +4,5 @@
         <sensor name="laser" type="ray">
             <pose>0 0 0 0 0 0</pose>
-            <visualize>true</visualize>
+            <visualize>false</visualize>
             <update_rate>10</update_rate>
             <ray>

File: src/diff_bot/urdf/links.urdf.xacro (robot description, xacro)
@@ -3,5 +3,5 @@
     <xacro:include filename="materials.xacro" />
     <xacro:include filename="inertia_macros.xacro" />
-    <link name="base_link" />
+    <link name="base_footprint" />
     <link name="chassis_link">
         <visual>

Commit message: SLAM works. navgitation does not work for goals that are far away - probably due to hardware limitations

File: src/diff_bot/urdf/diff_control.gazebo.xacro (robot description, xacro)
@@ -2,5 +2,5 @@
 <robot name="ultron" xmlns:xacro="http://www.ros.org/wiki/xacro">
     <gazebo>
-        <plugin name="diff_cont" filename="libgazebo_ros_diff_drive.so">
+        <plugin name="diff_controller" filename="libgazebo_ros_diff_drive.so">
             <left_joint>left_wheel_joint</left_joint>
             <right_joint>right_wheel_joint</right_joint>
@@ -10,5 +10,5 @@
             <max_wheel_acceleration>4</max_wheel_acceleration>
             <odometry_frame>odom</odometry_frame>
-            <ros_base_frame>base_footprint</ros_base_frame>
+            <robot_base_frame>base_link</robot_base_frame>
             <publish_odom>true</publish_odom>
             <publish_odom_tf>true</publish_odom_tf>

File: src/diff_bot/urdf/joints.urdf.xacro (robot description, xacro)
@@ -2,5 +2,5 @@
 <robot name="ultron" xmlns:xacro="http://www.ros.org/wiki/xacro">
     <joint name="chassis_joint" type="fixed">
-        <parent link="base_footprint" />
+        <parent link="base_link" />
         <child link="chassis_link" />
         <origin xyz="0 0 0.017" rpy="0 0 0" />

File: src/diff_bot/urdf/links.urdf.xacro (robot description, xacro)
@@ -3,5 +3,5 @@
     <xacro:include filename="materials.xacro" />
     <xacro:include filename="inertia_macros.xacro" />
-    <link name="base_footprint" />
+    <link name="base_link" />
     <link name="chassis_link">
         <visual>
